File: Hardware/Handheld.kicad_sch (KiCad schematic)
At the start: 7 parts, among them J1 USB_C_Receptacle_USB2.0_16P, U1 RASPBERRY_PI_ZERO_2_W, U2 BQ25308RTER

Commit message: ADC and Controls
Parts:
- removed R3: 10k, symbol Device:R
- removed U2: BQ25308RTER, WQFN16_RTE_TEX, symbol BQ25308:BQ25308RTER
Connections:
- net Battery Controller/VIN: now reaches J1.A4 (VBUS), J1.A9 (VBUS), J1.B4 (VBUS), J1.B9 (VBUS)
Other:
- added sheet Battery Controller (battery_controller.kicad_sch)
- added sheet Controls (controls.kicad_sch)
- moved on the sheet: BT1
