File: Hardware/controls.kicad_sch (KiCad schematic)
At the start: 7 parts, among them J2 Left Joystick, J3 Right Joystick, U2 ADS1115IDGSR

Commit message: In progress commit so that I can continue work on a different device
Parts:
- added R3, R5, R6: R, symbol Device:R
Connections:
- net +3.3V: now also U2.8 (VDD), R3.1, R5.1, R6.1
- net GND: now also U2.1 (ADDR), U2.3 (GND)
- net SCL: now reaches U2.10 (SCL)
- net SCL: now also R3.2
- net GPIO: now reaches U2.2 (ALERT/RDY)
- net GPIO: now also R6.2
- net SDA: now reaches U2.9 (SDA)
- net SDA: now also R5.2
Other:
- moved on the sheet: U2
